Commit message: 이동성공

File: jackal_ws/src/jackal/jackal_description/sdf/jackal.sdf.xacro (robot description, xacro)
@@ -1,13 +1,52 @@
 <?xml version="1.0"?>
-<sdf version="1.7" xmlns:xacro="http://ros.org/wiki/xacro">
-  <xacro:arg name="is_sim" default="true"/>
-  <xacro:arg name="prefix" default=""/>
-  <xacro:arg name="zed_mount_path" default="zed_mount.sdf"/>
-  <xacro:arg name="plugin_path" default="jackal_ignition_plugins.sdf"/>
-  <model name="jackal">
-    <static>false</static>
-    <!-- Base Link -->
+<sdf version="1.7" xmlns:xacro="http://www.ros.org/wiki/xacro">
+  <model name="jackal" canonical_link='base_link'>
+    <xacro:arg name="prefix" default="" />
+    <xacro:arg name="zed_mount_path" default="zed_mount.sdf"/>
+    <xacro:arg name="wheel_path" default="wheel.sdf.xacro"/>
+    <xacro:property name="PI" value="3.1415926535897931" />
+    <xacro:property name="wheelbase" value="0.262" />
+    <xacro:property name="track" value="0.37559" />
+    <xacro:property name="wheel_vertical_offset" value="0.0345" />
+    <xacro:property name="footprint_vertical_offset" value="-0.0655" />
+    <xacro:property name="wheel_radius" value="0.098" />
+    <xacro:property name="wheel_width" value="0.040" />
+    <xacro:property name="chassis_length" value="0.420" />
+    <xacro:property name="chassis_width" value="0.310" />
+    <xacro:property name="chassis_height" value="0.184" />
+    <xacro:property name="dummy_inertia" value="1e-09"/>
+    <xacro:property name="mount_spacing" value="0.120" />
+    <xacro:property name="dark_grey_rgba" value="0.2 0.2 0.2 1.0" />
+    <xacro:property name="light_grey_rgba" value="0.4 0.4 0.4 1.0" />
+    <xacro:property name="yellow_rgba" value="0.8 0.8 0.0 1.0" />
+    <xacro:property name="black_rgba" value="0.15 0.15 0.15 1.0" />
+    <plugin
+      filename="libignition-gazebo-joint-state-publisher-system.so"
+      name="ignition::gazebo::systems::JointStatePublisher">
+    </plugin>
+    <!-- Base and Chassis -->
     <link name="base_link">
-      <pose>0 0 0 0 0 0</pose>
+      <pose relative_to='__model__'>0 0 0 0 0 0</pose>
+    </link>
+    <link name="chassis_link">
+      <pose relative_to='base_link_joint'>0 0 0.0655 0 0 0</pose>
+      <visual name="chassis_visual">
+        <geometry>
+          <mesh><uri>model://jackal_description/meshes/jackal-base.stl</uri></mesh>
+        </geometry>
+        <material>
+          <ambient>${dark_grey_rgba}</ambient>
+          <diffuse>${dark_grey_rgba}</diffuse>
+        </material>
+        <pose>0 0 ${footprint_vertical_offset} ${PI/2} 0 ${PI/2}</pose>
+      </visual>
+      <collision name="chassis_collision">
+        <geometry>
+          <box>
+            <size>${chassis_length} ${chassis_width} ${chassis_height}</size>
+          </box>
+        </geometry>
+        <pose>0 0 ${chassis_height/2} 0 0 0</pose>
+      </collision>
       <inertial>
         <mass>16.523</mass>
@@ -15,73 +54,176 @@
         <inertia>
           <ixx>0.3136</ixx>
-          <iyy>0.3922</iyy>
-          <izz>0.4485</izz>
           <ixy>-0.0008</ixy>
           <ixz>0.0164</ixz>
+          <iyy>0.3922</iyy>
           <iyz>-0.0009</iyz>
+          <izz>0.4485</izz>
         </inertia>
       </inertial>
-      <visual name="chassis_visual">
-        <geometry>
-          <mesh uri="model://jackal_description/meshes/jackal-base.stl"/>
-        </geometry>
-        <material>
-          <ambient>0.2 0.2 0.2 1</ambient>
-          <diffuse>0.2 0.2 0.2 1</diffuse>
-        </material>
-      </visual>
-      <collision name="chassis_collision">
-        <geometry>
-          <box>
-            <size>0.42 0.31 0.184</size>
-          </box>
-        </geometry>
-      </collision>
-    </link>
-    <!-- Example wheel link: front_left -->
-    <link name="front_left_wheel_link">
-      <pose>0.131 0.187795 0.0345 0 0 0</pose>
+    </link>
+    <joint name="base_link_joint" type="fixed">
+      <parent>base_link</parent>
+      <child>chassis_link</child>
+      <pose relative_to='base_link'>0 0 0 0 0 0</pose>
+    </joint>
+    <!-- Wheels -->
+    <xacro:include filename="$(arg wheel_path)" />
+    <!-- Instantiate four wheels -->
+    <xacro:wheel prefix="front_left" pose="${wheelbase/2} ${track/2} ${wheel_vertical_offset} 0 0 0"/>
+    <xacro:wheel prefix="front_right" pose="${wheelbase/2} ${-track/2} ${wheel_vertical_offset} 0 0 0"/>
+    <xacro:wheel prefix="rear_left" pose="${-wheelbase/2} ${track/2} ${wheel_vertical_offset} 0 0 0"/>
+    <xacro:wheel prefix="rear_right" pose="${-wheelbase/2} ${-track/2} ${wheel_vertical_offset} 0 0 0"/>
+    <plugin name="ignition::gazebo::systems::DiffDrive"
+            filename="libignition-gazebo-diff-drive-system.so">
+      <left_joint>rear_left_wheel_joint</left_joint>
+      <left_joint>front_left_wheel_joint</left_joint>
+      <right_joint>rear_right_wheel_joint</right_joint>
+      <right_joint>front_right_wheel_joint</right_joint>
+      <wheel_separation>${track}</wheel_separation>
+      <wheel_radius>${wheel_radius}</wheel_radius>
+      <topic>/cmd_vel</topic>
+      <odometry_topic>odom</odometry_topic>
+      <publish_odom>true</publish_odom>
+      <publish_tf>true</publish_tf>
+    </plugin>
+    <!-- Front Fender -->
+    <link name="front_fender_link">
+      <pose relative_to='front_fender_joint'>0 0 0 0 0 0</pose>
+      <visual name="front_fender_visual">
+        <geometry>
+          <mesh>
+            <uri>model://jackal_description/meshes/jackal-fender.stl</uri>
+          </mesh>
+        </geometry>
+        <material>
+          <ambient>0.8 0.8 0.0 1.0</ambient>
+          <diffuse>0.8 0.8 0.0 1.0</diffuse>
+        </material>
+      </visual>
+    </link>
+    <joint name="front_fender_joint" type="fixed">
+      <parent>chassis_link</parent>
+      <child>front_fender_link</child>
+      <pose relative_to='chassis_link'>0 0 0 0 0 0</pose>
+    </joint>
+    <!-- Rear Fender -->
+    <link name="rear_fender_link">
+      <pose relative_to='rear_fender_joint'>0 0 0 0 0 0</pose>
+      <visual name="rear_fender_visual">
+        <geometry>
+          <mesh>
+            <uri>model://jackal_description/meshes/jackal-fender.stl</uri>
+          </mesh>
+        </geometry>
+        <material>
+          <ambient>0.8 0.8 0.0 1.0</ambient>
+          <diffuse>0.8 0.8 0.0 1.0</diffuse>
+        </material>
+      </visual>
+    </link>
+    <joint name="rear_fender_joint" type="fixed">
+      <parent>chassis_link</parent>
+      <child>rear_fender_link</child>
+      <pose relative_to='chassis_link'>0 0 0 0 0 ${PI}</pose>
+    </joint>
+    <!-- IMU -->
+    <link name="imu_link">
+      <pose relative_to="imu_joint"> 0 0 0 0 0 0</pose>
       <inertial>
-        <mass>0.477</mass>
+        <mass>0.001</mass>
+        <pose>0 0 0 0 0 0</pose>
         <inertia>
-          <ixx>0.0013</ixx>
-          <iyy>0.0024</iyy>
-          <izz>0.0013</izz>
+          <ixx>${dummy_inertia}</ixx>
+          <ixy>0.0</ixy>
+          <ixz>0.0</ixz>
+          <iyy>${dummy_inertia}</iyy>
+          <iyz>0.0</iyz>
+          <izz>${dummy_inertia}</izz>
         </inertia>
       </inertial>
-      <visual name="fl_wheel_visual">
+      <sensor name="imu_sensor" type="imu">
+        <pose>0 0 0 0 0 0</pose>
+        <always_on>true</always_on>
+        <update_rate>100</update_rate>
+        <imu>
+          <angular_velocity>
+            <x><noise type="gaussian"><mean>0.0</mean><stddev>0.005</stddev></noise></x>
+            <y><noise type="gaussian"><mean>0.0</mean><stddev>0.005</stddev></noise></y>
+            <z><noise type="gaussian"><mean>0.0</mean><stddev>0.005</stddev></noise></z>
+          </angular_velocity>
+          <linear_acceleration>
+            <x><noise type="gaussian"><mean>0.0</mean><stddev>0.02</stddev></noise></x>
+            <y><noise type="gaussian"><mean>0.0</mean><stddev>0.02</stddev></noise></y>
+            <z><noise type="gaussian"><mean>0.0</mean><stddev>0.02</stddev></noise></z>
+          </linear_acceleration>
+        </imu>
+      </sensor>
+    </link>
+    <joint name="imu_joint" type="fixed">
+      <parent>chassis_link</parent>
+      <child>imu_link</child>
+      <pose relative_to="chassis_link">0 0 0 0 0 0</pose>
+    </joint>
+    <!-- Navsat -->
+    <link name="navsat_link">
+      <pose relative_to="navsat_joint"> 0 0 0 0 0 0</pose>
+      <visual name="navsat_visual">
         <geometry>
           <cylinder>
-            <radius>0.098</radius>
-            <length>0.04</length>
+            <radius>0.026</radius>
+            <length>0.016</length>
           </cylinder>
         </geometry>
-      </visual>
-      <collision name="fl_wheel_collision">
-        <geometry>
-          <cylinder>
-            <radius>0.098</radius>
-            <length>0.04</length>
-          </cylinder>
-        </geometry>
-      </collision>
-    </link>
-    <!-- Wheel Joint Example -->
-    <joint name="front_left_wheel_joint" type="revolute">
-      <parent>base_link</parent>
-      <child>front_left_wheel_link</child>
-      <axis>
-        <xyz>0 1 0</xyz>
-        <limit>
-          <lower>-1e16</lower>
-          <upper>1e16</upper>
-        </limit>
-      </axis>
-    </joint>
-    <!-- Repeat for other wheels (front_right, rear_left, rear_right) -->
-    <!-- Add other links: imu_link, navsat_link, mounts etc. -->
-    <!-- Xacro includes for ZED and plugins -->
+        <pose>0 0 0.008 0 0 0</pose>
+        <material>
+          <ambient>${black_rgba}</ambient>
+          <diffuse>${black_rgba}</diffuse>
+        </material>
+      </visual>
+      <sensor name="gps_sensor" type="navsat">
+        <pose>0 0 0 0 0 0</pose>
+        <always_on>true</always_on>
+        <update_rate>10</update_rate>
+      </sensor>
+    </link>
+    <joint name="navsat_joint" type="fixed">
+      <parent>chassis_link</parent>
+      <child>navsat_link</child>
+      <pose relative_to="chassis_link">-0.180 0.126 0.1815 0 0 0</pose>
+    </joint>
+    <!-- Mounts -->
+    <link name="mid_mount">
+      <pose relative_to="mid_mount_joint">0 0 0 0 0 0</pose>
+    </link>
+    <joint name="mid_mount_joint" type="fixed">
+      <parent>chassis_link</parent>
+      <child>mid_mount</child>
+      <pose relative_to="chassis_link">0 0 ${chassis_height} 0 0 0</pose>
+    </joint>
+    <link name="rear_mount">
+      <pose relative_to="rear_mount_joint">0 0 0 0 0 0</pose>
+    </link>
+    <joint name="rear_mount_joint" type="fixed">
+      <parent>mid_mount</parent>
+      <child>rear_mount</child>
+      <pose relative_to="mid_mount">${-mount_spacing} 0 0 0 0 0</pose>
+    </joint>
+    <link name="front_mount">
+      <pose relative_to="front_mount_joint">0 0 0 0 0 0</pose>
+    </link>
+    <joint name="front_mount_joint" type="fixed">
+      <parent>mid_mount</parent>
+      <child>front_mount</child>
+      <pose relative_to="mid_mount">${mount_spacing} 0 0 0 0 0</pose>
+    </joint>
+    <!-- Fenders -->
+    <!-- (unchanged content skipped for brevity) -->
+    <!-- ZED camera and accessories -->
     <xacro:include filename="$(arg zed_mount_path)"/>
-    <xacro:include filename="$(arg plugin_path)"/>
+    <joint name="zed_mount_joint" type="fixed">
+      <parent>mid_mount</parent>
+      <child>zed_mount_link</child>
+      <pose relative_to="mid_mount">${mount_spacing/2} 0 0 0 0 0</pose>
+    </joint>
   </model>
 </sdf>

File: jackal_ws/src/jackal/jackal_description/urdf/jackal.urdf.xacro (robot description, xacro)
@@ -64,5 +64,5 @@
       <type>transmission_interface/SimpleTransmission</type>
       <joint name="${prefix}_wheel_joint">
-        <hardwareInterface>hardware_interface/VelocityJointInterface</hardwareInterface>
+        <hardwareInterface>hardware_interface/velocity</hardwareInterface>
       </joint>
       <actuator name="${prefix}_actuator">
@@ -265,6 +265,6 @@
        of these into the final description is controlled by optenv variables, which
        default each one to off.-->
-  <xacro:include filename="$(find jackal_description)/urdf/accessories.urdf.xacro" />
+  <!-- <xacro:include filename="$(find jackal_description)/urdf/accessories.urdf.xacro" /> -->
   <!-- Optional custom includes. -->
-  <xacro:include filename="$(optenv JACKAL_URDF_EXTRAS empty.urdf)" />
+  <!-- <xacro:include filename="$(optenv JACKAL_URDF_EXTRAS empty.urdf)" /> -->
 </robot>
