Commit message: 5/12-밭 최적화밑 gps localization 수정중

File: jackal_ws/src/jackal/jackal_description/urdf/custom_zed_mount.urdf.xacro (robot description, xacro)
@@ -8,5 +8,7 @@
       </geometry>
       <origin xyz="0 0 0" rpy="${PI/2} 0 ${PI/2}"/>
-      <material name="light_grey" />
+      <material name="light_grey">
+        <color rgba="0.4 0.4 0.4 1.0" />
+      </material>
     </visual>
     <collision>
@@ -28,4 +30,8 @@
     </inertial>
   </link>
+  <gazebo reference="zed_mount_link">
+    <material>Gazebo/Grey</material>
+    <turnGravityOff>false</turnGravityOff>
+  </gazebo>
   <joint name="zed_mount_joint" type="fixed">
     <parent link="mid_mount"/>  <!-- 또는 front_mount, rear_mount 등 위치 선택 -->
@@ -40,5 +46,7 @@
       </geometry>
       <origin xyz="-0.036262 0.008969 0.017741" rpy="0 0 ${PI/2}"/>
-      <material name="black" />
+      <material name="black">
+        <color rgba="0.15 0.15 0.15 1.0" />
+      </material>
     </visual>
     <collision>
@@ -61,4 +69,8 @@
     </inertial>
   </link>
+  <gazebo reference="zed_2i_link">
+    <material>Gazebo/Black</material>
+    <turnGravityOff>false</turnGravityOff>
+  </gazebo>
   <joint name="zed_2i_base_joint" type="fixed">
     <parent link="zed_mount_link"/>
@@ -104,8 +116,8 @@
           <width>1280</width>
           <height>960</height>
-          <format>B8G8R8</format>
+          <format>R8G8B8</format>
         </image>
         <clip>
-          <near>0.1</near>
+          <near>0.03</near>
           <far>20.0</far>
         </clip>

File: jackal_ws/src/jackal/jackal_description/urdf/jackal.urdf.xacro (robot description, xacro)
@@ -45,9 +45,8 @@
     </link>
     <gazebo reference="${prefix}_wheel_link">
-      <material>Gazebo/DarkGrey</material>
+      <material>Gazebo/Black</material>
       <selfCollide>false</selfCollide>
       <mu1 value="0.5"/>
       <mu2 value="0.5"/>
-      <fdir1>1 0 0</fdir1>
       <kp value="10000000.0" />
       <kd value="1" />
@@ -58,7 +57,5 @@
       <child link="${prefix}_wheel_link" />
       <xacro:insert_block name="joint_pose" />
-      <axis xyz="0 1 0">
-        <dynamics damping="1.0" friction="0.0"/>
-      </axis>
+      <axis xyz="0 1 0"/>
     </joint>
     <!-- In reality, Jackal has only two motors, one per side. However, it's more
@@ -193,4 +190,5 @@
     <parent link="chassis_link" />
     <child link="imu_link" />
+    <origin xyz="0 0 0" rpy="0 0 0"/>
   </joint>
   <!-- TODO: Same note as applies to imu_link -->
