Commit message: 월드구현 토마토밭

File: jackal_ws/src/jackal/jackal_description/urdf/jackal.urdf.xacro (robot description, xacro)
@@ -49,4 +49,5 @@
       <mu1 value="0.5"/>
       <mu2 value="0.5"/>
+      <fdir1>1 0 0</fdir1>
       <kp value="10000000.0" />
       <kd value="1" />
@@ -57,5 +58,7 @@
       <child link="${prefix}_wheel_link" />
       <xacro:insert_block name="joint_pose" />
-      <axis xyz="0 1 0" />
+      <axis xyz="0 1 0">
+        <dynamics damping="1.0"/>
+      </axis>
     </joint>
     <!-- In reality, Jackal has only two motors, one per side. However, it's more

Commit message: slam성공밑 navigation이동 이상한거 해결중

File: jackal_ws/src/jackal/jackal_description/urdf/jackal.urdf.xacro (robot description, xacro)
@@ -59,5 +59,5 @@
       <xacro:insert_block name="joint_pose" />
       <axis xyz="0 1 0">
-        <dynamics damping="1.0"/>
+        <dynamics damping="1.0" friction="0.0"/>
       </axis>
     </joint>

Commit message: gps localization완료

File: jackal_ws/src/jackal/jackal_description/urdf/jackal.urdf.xacro (robot description, xacro)
@@ -198,5 +198,5 @@
         <cylinder radius="0.026" length="0.016" />
       </geometry>
-      <origin xyz="0 0 0.008" />
+      <origin xyz="-0.180 0.126 0.1895" />
       <material name="black" />
     </visual>
@@ -205,5 +205,5 @@
     <parent link="chassis_link" />
     <child link="navsat_link" />
-    <origin xyz="-0.180 0.126 0.1815" />
+    <origin xyz="0 0 0" />
   </joint>
   <link name="mid_mount"></link>
