Commit message: navigation 최적화(lidar추가+속도 높임+파라미터 수정))

File: jackal_ws/src/jackal/jackal_description/urdf/custom_mount.urdf.xacro (robot description, xacro)
@@ -1,4 +1,58 @@
 <?xml version="1.0"?>
 <robot xmlns:xacro="http://www.ros.org/wiki/xacro">
+  <link name="lidar_link">
+    <visual>
+      <geometry><cylinder radius="0.05" length="0.05"/></geometry>
+      <origin xyz="0 0 0.025" />
+      <material name="black" />
+    </visual>
+    <collision>
+      <geometry><cylinder radius="0.05" length="0.05"/></geometry>
+    </collision>
+    <inertial>
+      <mass value="0.1"/>
+      <origin xyz="0 0 0" rpy="0 0 0"/>
+      <inertia
+        ixx="0.0001" ixy="0.0"  ixz="0.0"
+        iyy="0.0001" iyz="0.0"
+        izz="0.0001"/>
+    </inertial>
+  </link>
+  <joint name="lidar_joint" type="fixed">
+    <parent link="front_mount"/>
+    <child link="lidar_link"/>
+    <origin xyz="0.06 0 0" rpy="0 0 0"/>
+  </joint>
+  <gazebo reference="lidar_link">
+    <sensor name="lidar" type="ray">
+      <ray>
+        <scan>
+          <horizontal>
+            <samples>720</samples>
+            <resolution>1</resolution>
+            <min_angle>-1.57</min_angle>
+            <max_angle>1.57</max_angle>
+          </horizontal>
+        </scan>
+        <range>
+          <min>0.1</min>
+          <max>10.0</max>
+        </range>
+      </ray>
+      <plugin name="gazebo_ros_laser_controller" filename="libgazebo_ros_ray_sensor.so">
+        <ros>
+          <remapping>~/out:=/scan</remapping>
+        </ros>
+        <frame_name>lidar_link</frame_name>
+        <topic_name>/scan</topic_name>
+        <output_type>sensor_msgs/LaserScan</output_type>
+      </plugin>
+      <always_on>true</always_on>
+      <update_rate>10.0</update_rate>
+      <visualize>false</visualize>
+    </sensor>
+    <material>Gazebo/Black</material>
+    <turnGravityOff>false</turnGravityOff>
+  </gazebo>
   <!-- 지지대 링크 -->
   <link name="zed_mount_link">

File: jackal_ws/src/jackal/jackal_description/urdf/jackal.urdf.xacro (robot description, xacro)
@@ -262,5 +262,5 @@
   </xacro:if>
   <!-- 우리 프로젝트에 필요한 zed카메라 장착 -->
-  <xacro:include filename="$(find jackal_description)/urdf/custom_zed_mount.urdf.xacro"/>
+  <xacro:include filename="$(find jackal_description)/urdf/custom_mount.urdf.xacro"/>
   <!-- Optional standard accessories, including their simulation data. The rendering
        of these into the final description is controlled by optenv variables, which
