Commit message: description/ golbal pose / move_to_goal_action
nav2랑 merged하고 , 노드 수정한 commit

File: jackal_ws/src/jackal/jackal_description/urdf/jackal.urdf (robot description, URDF)
Before this commit: robot jackal, 19 links, 18 joints
Joints:
- joint imu_joint: origin (none) -> xyz=0 0 0 rpy=0 0 0

Commit message: [feat] ActionLancher

File: jackal_ws/src/jackal/jackal_description/urdf/jackal.urdf (robot description, URDF)
Before this commit: robot jackal, 19 links, 18 joints
Joints:
- joint navsat_joint: origin xyz=-0.180 0.126 0.1815 -> xyz=0 0 0

Commit message: [chore] Twist Mux 다시 추가

File: jackal_ws/src/jackal/jackal_description/urdf/jackal.urdf (robot description, URDF)
Before this commit: robot jackal, 19 links, 18 joints
Links:
- added link lidar_link, mass 0.1; collision cylinder length=0.05 radius=0.05; visual cylinder length=0.05 radius=0.05
Joints:
- added joint lidar_joint: type fixed, parent front_mount, child lidar_link, origin xyz=0.06 0 0 rpy=0 0 0
